Commit message: Readme update, typo

File: src/myrobot_description/urdf/robot.xacro (robot description, xacro)
@@ -111,5 +111,5 @@
     </link>
     <!--  Base footprint -->
-    <link name="base_footprint"/ode to publish th>
+    <link name="base_footprint"/>
     <!-- Base footprint joint -->
     <joint name="base_footprint_joint" type="fixed">

Commit message: added robot yaml importing

File: src/myrobot_description/urdf/robot.xacro (robot description, xacro)
@@ -2,4 +2,6 @@
 <robot name="differential_drive_robot" xmlns:xacro="http://www.ros.org/wiki/xacro">
     <xacro:include filename="$(find myrobot_description)/urdf/include/inertial.xacro" />
+    <!-- <xacro:property name="robot_yaml" value="$(find myrobot_description)/config/robot.yaml" />
+    <xacro:property name="robot" value="${xacro.load_yaml(robot_yaml)}"/> -->
     <!-- Robot Parameters -->
     <xacro:property name="body_length" value="0.45"/>
