Commit message: Added my changes from local ros2workshop folder

File: src/myrobot_description/urdf/robot.urdf.xacro (robot description, xacro)
@@ -188,3 +188,7 @@
             rpy="${sensors['camera']['roll']} ${sensors['camera']['pitch']} ${sensors['camera']['yaw']}" />
     </xacro:camera>
+    <xacro:lidar lidar="${sensors['lidar']}" robot="myrobot">
+        <origin xyz="${sensors['lidar']['x']} ${sensors['lidar']['y']} ${sensors['lidar']['z']}"
+            rpy="${sensors['lidar']['roll']} ${sensors['lidar']['pitch']} ${sensors['lidar']['yaw']}" />
+    </xacro:lidar>
 </robot>
