Commit message: added camera

File: src/myrobot_description/urdf/include/sensors_macros.xacro (robot description, xacro)
@@ -2,4 +2,69 @@
 <robot xmlns:xacro="http://www.ros.org/wiki/xacro">
     <!-- Camera -->
+    <xacro:macro name="camera" params=" *joint_origin camera robot">
+        <link name="${camera['name']}_link">
+            <collision>
+                <origin xyz="0 0 0" rpy="0 ${pi/2} 0"/>
+                <geometry>
+                    <cylinder radius="${camera['radius']}" length="${camera['length']}"/>
+                </geometry>
+            </collision>
+            <visual>
+                <origin xyz="0 0 0" rpy="0 ${pi/2} 0"/>
+                <geometry>
+                    <cylinder radius="${camera['radius']}" length="${camera['length']}"/>
+                <!-- TODO add mesh insertion capabilities -->
+                </geometry>
+            </visual>
+            <inertial>
+                <mass value="1e-5" />
+                <origin xyz="0 0 0" rpy="0 0 0"/>
+                <inertia ixx="1e-6" ixy="0" ixz="0" iyy="1e-6" iyz="0" izz="1e-6" />
+            </inertial>
+        </link>
+        <joint name="${camera['name']}_joint" type="fixed">
+            <axis xyz="0 1 0" />
+            <xacro:insert_block name="joint_origin" />
+            <parent link="${camera['parent_link']}"/>
+            <child link="${camera['name']}_link"/>
+        </joint>
+        <gazebo reference="${camera['name']}_link">
+            <material>Gazebo/Red</material>
+        </gazebo>
+        <gazebo reference="${camera['name']}_link">
+            <sensor type="camera" name="${camera['name']}">
+                <topic>${camera['image_topic']}</topic>
+                <update_rate>${camera['update_rate']}</update_rate>
+                <visualize>${camera['cam_view_visualize']}</visualize>
+                <camera>
+                    <horizontal_fov>${camera['horizontal_fov']}</horizontal_fov>
+                    <image>
+                        <width>${camera['width']}</width>
+                        <height>${camera['height']}</height>
+                        <format>${camera['format']}</format>
+                    </image>
+                    <clip>
+                        <near>0.02</near>
+                        <far>300</far>
+                    </clip>
+                    <noise>
+                    <type>gaussian</type>
+                    <!-- Noise is sampled independently per pixel on each frame.
+                            That pixel's noise value is added to each of its color
+                            channels, which at that point lie in the range [0,1]. -->
+                    <mean>0.0</mean>
+                    <stddev>0.007</stddev>
+                    </noise>
+                    <camera_info_topic>${camera['info_topic']}</camera_info_topic>
+                </camera>
+                <plugin filename="gz-sim-sensors-system" name="gz::sim::systems::Sensors">
+                    <always_on>true</always_on>
+                    <visualize>true</visualize>
+                    <update_rate>30</update_rate>
+                    <gz_frame_id>camera_rgb_frame</gz_frame_id>
+                </plugin>
+            </sensor>
+        </gazebo>
+    </xacro:macro>
     <!-- Lidar -->
 </robot>

File: src/myrobot_description/urdf/robot.urdf.xacro (robot description, xacro)
@@ -4,4 +4,7 @@
     <!-- <xacro:property name="robot_yaml" value="$(find myrobot_description)/config/robot.yaml" />
     <xacro:property name="robot" value="${xacro.load_yaml(robot_yaml)}"/> -->
+    <xacro:include filename="$(find myrobot_description)/urdf/include/sensors_macros.xacro" />
+    <xacro:property name="sensors_yaml" value="$(find myrobot_description)/config/sensors.yaml" />
+    <xacro:property name="sensors" value="${xacro.load_yaml(sensors_yaml)}"/>
     <!-- Robot Parameters -->
     <xacro:property name="body_length" value="0.45"/>
@@ -180,3 +183,7 @@
         </plugin>
     </gazebo>
+    <xacro:camera camera="${sensors['camera']}" robot="myrobot">
+        <origin xyz="${sensors['camera']['x']} ${sensors['camera']['y']} ${sensors['camera']['z']}"
+            rpy="${sensors['camera']['roll']} ${sensors['camera']['pitch']} ${sensors['camera']['yaw']}" />
+    </xacro:camera>
 </robot>

Commit message: Added lidar plugin

File: src/myrobot_description/urdf/include/sensors_macros.xacro (robot description, xacro)
@@ -1,6 +1,9 @@
 <?xml version="1.0"?>
 <robot xmlns:xacro="http://www.ros.org/wiki/xacro">
+    <gazebo>
+        <plugin filename="gz-sim-sensors-system" name="gz::sim::systems::Sensors"/>
+    </gazebo>
     <!-- Camera -->
-    <xacro:macro name="camera" params=" *joint_origin camera robot">
+    <xacro:macro name="camera" params="*joint_origin camera robot">
         <link name="${camera['name']}_link">
             <collision>
@@ -36,5 +39,5 @@
                 <topic>${camera['image_topic']}</topic>
                 <update_rate>${camera['update_rate']}</update_rate>
-                <visualize>${camera['cam_view_visualize']}</visualize>
+                <gz_frame_id>${camera['frame_name']}</gz_frame_id>
                 <camera>
                     <horizontal_fov>${camera['horizontal_fov']}</horizontal_fov>
@@ -58,13 +61,70 @@
                     <camera_info_topic>${camera['info_topic']}</camera_info_topic>
                 </camera>
-                <plugin filename="gz-sim-sensors-system" name="gz::sim::systems::Sensors">
-                    <always_on>true</always_on>
-                    <visualize>true</visualize>
-                    <update_rate>30</update_rate>
-                    <gz_frame_id>camera_rgb_frame</gz_frame_id>
-                </plugin>
+                <visualize>true</visualize>
             </sensor>
         </gazebo>
     </xacro:macro>
     <!-- Lidar -->
+    <xacro:macro name="lidar" params="*joint_origin lidar robot">
+        <link name="${lidar['name']}_link">
+            <collision>
+                <origin xyz="0 0 0" rpy="0 0 0"/>
+                <geometry>
+                    <cylinder radius="${lidar['radius']}" length="${lidar['length']}"/>
+                </geometry>
+            </collision>
+            <visual>
+                <origin xyz="0 0 0" rpy="0 0 0"/>
+                <geometry>
+                    <cylinder radius="${lidar['radius']}" length="${lidar['length']}"/>
+                <!-- TODO add mesh insertion capabilities -->
+                </geometry>
+            </visual>
+            <inertial>
+                <mass value="1e-5" />
+                <origin xyz="0 0 0" rpy="0 0 0"/>
+                <inertia ixx="1e-6" ixy="0" ixz="0" iyy="1e-6" iyz="0" izz="1e-6" />
+            </inertial>
+        </link>
+        <joint name="${lidar['name']}_joint" type="fixed">
+            <axis xyz="0 1 0" />
+            <xacro:insert_block name="joint_origin" />
+            <parent link="${lidar['parent_link']}"/>
+            <child link="${lidar['name']}_link"/>
+        </joint>
+        <gazebo reference="${lidar['name']}_link">
+            <material>Gazebo/Blue</material>
+        </gazebo>
+        <gazebo reference="${lidar['name']}_link">
+            <sensor name='lidar' type='gpu_lidar'>
+                <always_on>true</always_on>
+                <visualize>true</visualize>
+                <pose>0 0 0 0 0 0</pose>
+                <topic>${lidar['topic']}</topic>
+                <update_rate>${lidar['update_rate']}</update_rate>
+                <gz_frame_id>lidar_link</gz_frame_id>
+                <ray>
+                    <scan>
+                        <horizontal>
+                            <samples>${lidar['samples']}</samples>
+                            <resolution>${lidar['resolution']}</resolution>
+                            <min_angle>${lidar['min_angle']}</min_angle>
+                            <max_angle>${lidar['max_angle']}</max_angle>
+                        </horizontal>
+                        <vertical>
+                            <samples>1</samples>
+                            <resolution>0.01</resolution>
+                            <min_angle>0</min_angle>
+                            <max_angle>0</max_angle>
+                        </vertical>
+                    </scan>
+                    <range>
+                        <min>${lidar['min_range']}</min>
+                        <max>${lidar['max_range']}</max>
+                        <resolution>0.01</resolution>
+                    </range>
+                </ray>
+            </sensor>
+        </gazebo>
+    </xacro:macro>
 </robot>
